Commit message: committing changes

File: description/urdf/pioneer3at.urdf.xacro (robot description, xacro)
@@ -5,35 +5,6 @@
        xmlns:xacro="http://ros.org/wiki/xacro"
 name="pioneer3at">
-<gazebo>
-    <plugin name="gazebo_ros_control" filename="libgazebo_ros_control.so">
-      <robotNamespace>/rrbot</robotNamespace>
-      <robotSimType>gazebo_ros_control/DefaultRobotHWSim</robotSimType>
-    </plugin>
-  </gazebo>
-<xacro:include filename="$(find description)/urdf/pioneer3at.gazebo" />
-<!-- Chassis -->
-	<link name="base_link">
-		<!--  For pointers on inertial and gazebo-related parameters see
-		       * http://wiki.ros.org/urdf/Tutorials/Adding%20Physical%20and%20Collision%20Properties%20to%20a%20URDF%20Model
-                       * http://answers.gazebosim.org/question/4372/the-inertia-matrix-explained/
-		       * http://gazebosim.org/tutorials?tut=inertia&cat=build_robot, and
-                       * http://gazebosim.org/tutorials/?tut=ros_urdf
-                       * http://en.wikipedia.org/wiki/List_of_moment_of_inertia_tensors
-                -->
-		<inertial>
-			<mass value="21.5"/> <!-- P3AT 18.6kg plus three batteries @ 2.4kg each  minus four wheels @ 1.4 kg ea and top plate @ 0.1 kg-->
-			<origin xyz="0 -0.1 0.177"/>
-			<inertia ixx="0.3338" ixy="0.0"     ixz="0.0"
-				              iyy="0.4783"  iyz="0.0"
-				                            izz="0.3338"/>
-		</inertial>
-		<visual name="base_visual">
-			<origin xyz="0 0 0.177" rpy="0 0 0"/>
-			<geometry name="pioneer_geom">
-				<mesh filename="package://amr_robots_description/meshes/p3at_meshes/chassis.stl"/>
-			</geometry>
-			<material name="ChassisRed"/>
-		</visual>
-		<collision>
+    <link name="base_link">
+ <collision>
 			<origin xyz="0 0 0.177" rpy="0 0 0"/>
 				<geometry>
@@ -41,4 +12,435 @@
 				</geometry>
 		</collision>
-	</link>
+    <visual>
+    <origin xyz="0 0 0.177" rpy="0 0 0"/>
+	<geometry>
+        <mesh filename="package://amr_robots_description/meshes/p3at_meshes/chassis.stl"/>
+      </geometry>
+    </visual>
+<inertial>
+			<mass value="21.5"/> <!-- P3AT 18.6kg plus three batteries @ 2.4kg each  minus four wheels @ 1.4 kg ea and top plate @ 0.1 kg-->
+			<origin xyz="0 -0.1 0.177"/>
+			<inertia ixx="0.3338" ixy="0.0" ixz="0.0" iyy="0.4783" iyz="0.0" izz="0.3338"/>
+</inertial>
+  </link>
+  <gazebo reference="base_link">
+<material>Gazebo/Orange</material>
+  </gazebo>
+  <joint name="imu_joint" type="fixed">
+    <axis xyz="1 0 0"/> <!-- 0 1 0 -->
+    <origin xyz="0 0 0.19"/>
+    <parent link="base_link"/>
+    <child link="imu_link"/>
+  </joint>
+  <joint name="basefootprint_joint" type="fixed">
+    <axis xyz="1 0 0"/> <!-- 0 1 0 -->
+    <origin xyz="0 0 0.19"/>
+    <parent link="base_link"/>
+    <child link="base_footprint"/>
+  </joint>
+<link name="base_footprint">
+  <visual>
+    <origin rpy="0 0 0" xyz="0 0 0"/>
+    <geometry>
+      <box size="0.001 0.001 0.001"/>
+    </geometry>
+  </visual>
+</link>
+<link name="imu_link">
+   <collision>
+    <origin rpy="0 0 0" xyz="0 0 0"/>
+    <geometry>
+      <box size=".001 .001 .001"/>
+    </geometry>
+  </collision>
+  <visual>
+    <origin rpy="0 0 0" xyz="0 0 0"/>
+    <geometry>
+      <box size="0.001 0.001 0.001"/>
+    </geometry>
+  </visual>
+   <inertial>
+    <mass value="0.001"/>
+    <origin rpy="0 0 0" xyz="0 0 0"/>
+    <inertia ixx="0.0001" ixy="0" ixz="0" iyy="0.000001" iyz="0" izz="0.0001"/>
+  </inertial>
+</link>
+<!-- Top -->
+    <joint name="base_top_joint" type="fixed">
+		<origin xyz="0.003 0 0.274" rpy="0 0 0"/>
+		<parent link="base_link"/>
+		<child link="top_plate"/>
+	</joint>
+	<link name="top_plate">
+		<collision>
+			<origin xyz="0 0 0" rpy="0 0 0"/>
+			<geometry>
+				<box size="0.1 0.1 0.1"/>
+			</geometry>
+		</collision>
+		<visual>
+			<origin xyz="0 0 0" rpy="0 0 0"/>
+			<geometry>
+				<mesh filename="package://amr_robots_description/meshes/p3at_meshes/top.stl"/>
+			</geometry>
+		</visual>
+		<inertial>
+			<mass value="0.1"/>
+			<origin xyz="-0.025 0 -0.223"/>
+			<inertia ixx="1.0" ixy="0.0" ixz="0.0" iyy="1.0" iyz="0.0" izz="1.0"/>
+		</inertial>
+	</link>
+	<gazebo reference="top_plate">
+    <material>Gazebo/Blue</material>
+	</gazebo>
+<!-- Front + Back Sonar -->
+	<joint name="base_front_joint" type="fixed">
+		<origin xyz="0.193 0 0.25" rpy="0 0 0"/>
+		<parent link="base_link"/>
+		<child link="front_sonar"/>
+	</joint>
+	<link name="front_sonar">
+		<collision>
+			<origin xyz="0 0 0" rpy="0 0 0"/>
+			<geometry>
+				<box size="0.1 0.1 0.1"/>
+			</geometry>
+		</collision>
+		<visual>
+			<origin xyz="0 0 0" rpy="0 0 0"/>
+			<geometry>
+				<mesh filename="package://amr_robots_description/meshes/p3at_meshes/front_sonar.stl"/>
+			</geometry>
+		</visual>
+		<inertial>
+			<mass value="0.1"/>
+			<origin xyz="0 0 0"/>
+			<inertia ixx="1.0" ixy="0.0" ixz="0.0" iyy="1.0" iyz="0.0" izz="1.0"/>
+		</inertial>
+	</link>
+    <gazebo reference="front_sonar">
+    <material>Gazebo/Yellow</material>
+	</gazebo>
+   <joint name="base_back_joint" type="fixed">
+		<origin xyz="-0.187 0 0.247" rpy="0 0 0"/>
+		<parent link="base_link"/>
+		<child link="back_sonar"/>
+	</joint>
+    <link name="back_sonar">
+		<collision>
+			<origin xyz="0 0 0" rpy="0 0 0"/>
+			<geometry>
+				<box size="0.1 0.1 0.1"/>
+			</geometry>
+		</collision>
+		<visual>
+			<origin xyz="0 0 0" rpy="0 0 0"/>
+			<geometry>
+				<mesh filename="package://amr_robots_description/meshes/p3at_meshes/back_sonar.stl"/>
+			</geometry>
+		</visual>
+		<inertial>
+			<mass value="0.1"/>
+			<origin xyz="0 0 0"/>
+			<inertia ixx="1.0" ixy="0.0" ixz="0.0" iyy="1.0" iyz="0.0" izz="1.0"/>
+		</inertial>
+	</link>
+	<gazebo reference="back_sonar">
+		<material>Gazebo/Yellow</material>
+	</gazebo>
+	<joint name="hokuyo_joint" type="fixed">
+		<axis xyz="0 1 0" />
+		<origin xyz="0 0 0.31" rpy="0 0 0"/>
+		<parent link="base_link"/>
+		<child link="hokuyo_link"/>
+	</joint>
+	<!-- Hokuyo Laser -->
+	<link name="hokuyo_link">
+		<collision>
+			<origin xyz="0 0 0" rpy="0 0 0"/>
+	      		<geometry>
+	    			<box size="0.1 0.1 0.1"/>
+	      		</geometry>
+	    	</collision>
+		<visual>
+			<origin xyz="0 0 0" rpy="0 0 0"/>
+		      	<geometry>
+				<mesh filename="package://amr_robots_description/meshes/p3at_meshes/hokuyo.dae"/>
+		      	</geometry>
+		</visual>
+		<inertial>
+	      		<mass value="1e-5" />
+	      		<origin xyz="0 0 0" rpy="0 0 0"/>
+	      		<inertia ixx="1e-6" ixy="0" ixz="0" iyy="1e-6" iyz="0" izz="1e-6" />
+	    	</inertial>
+	  </link>
+	<link name="hokuyo_scanLink">
+	</link>
+	<joint name="hokuyo_scanJoint" type="fixed">
+		<axis xyz="0 1 0" />
+		<origin xyz="0 0 0.03" rpy="0 0 0"/>
+		<parent link="hokuyo_link"/>
+		<child link="hokuyo_scanLink"/>
+	</joint>
+<xacro:macro name="p3at_drive_side" params="side reflect">
+  <!-- Front Axles + Wheels + Hubcaps -->
+	<link name="p3at_front_${side}_axle">
+		<inertial>
+			<mass value="0.1"/>
+			<origin xyz="0 0 0"/>
+			<inertia ixx="1.0" ixy="0.0" ixz="0.0"
+				 iyy="1.0" iyz="0.0" izz="1.0"/>
+  	 	</inertial>
+	<visual>
+		<origin xyz="0 0 0" rpy="0 0 0"/>
+		<geometry>
+			<mesh filename="package://amr_robots_description/meshes/p3at_meshes/axle.stl"/>
+		</geometry>
+	</visual>
+	<collision>
+		<origin xyz="0 0 0" rpy="0 0 0"/>
+		<geometry>
+			<box size="0.1 0.1 0.1"/>
+		</geometry>
+	</collision>
+	</link>
+	<gazebo reference="p3at_front_${side}_axle">
+		<material>Gazebo/Green</material>
+	</gazebo>
+	<joint name="base_front_${side}_axle_joint" type="fixed">
+		<origin xyz="0.135 ${reflect*0.156} 0.111" rpy="0 0 0"/>
+		<parent link="base_link"/>
+		<child link="p3at_front_${side}_axle"/>
+	</joint>
+	<link name="p3at_front_${side}_hub">
+		<inertial>
+			<mass value="0.1"/>
+			<origin xyz="0 0 0"/>
+			<inertia ixx="1.0" ixy="0.0" ixz="0.0"
+				 iyy="1.0" iyz="0.0" izz="1.0"/>
+  	 	</inertial>
+	<visual name="base_visual">
+		<origin xyz="0 0 0" rpy="0 0 0"/>
+		<geometry name="pioneer_geom">
+			<mesh filename="package://amr_robots_description/meshes/p3at_meshes/${side}_hubcap.stl"/>
+		</geometry>
+		<material name="HubcapYellow">
+			<color rgba="1.0 0.811 0.151 1.0"/>
+		</material>
+	</visual>
+	<collision>
+		<origin xyz="0 0 0" rpy="0 0 0"/>
+		<geometry>
+			<box size="0.1 0.1 0.1"/>
+		</geometry>
+	</collision>
+	</link>
+	<gazebo reference="p3at_front_${side}_hub">
+		<material value="Gazebo/Yellow"/>
+	</gazebo>
+	<joint name="base_front_${side}_hub_joint" type="fixed">
+		<origin xyz="0 ${reflect*0.041} 0" rpy="0 0 0"/>
+		<parent link="p3at_front_${side}_axle"/>
+		<child link="p3at_front_${side}_hub"/>
+	</joint>
+	<link name="p3at_front_${side}_wheel">
+		<inertial>
+			<mass value="1.2"/> <!-- 1.4 kg - axle 0.1 kg - hub 0.1 kg -->
+			<origin xyz="0 0 0"/>
+			<inertia ixx="0.012411765597" ixy="0" ixz="0"
+         iyy="0.015218160428" iyz="0" izz="0.011763977943"/>
+      </inertial>
+	<visual>
+		<origin xyz="0 0 0" rpy="0 0 0"/>
+		<geometry>
+			<mesh filename="package://amr_robots_description/meshes/p3at_meshes/wheel.stl"/>
+		</geometry>
+		<material name="WheelBlack">
+			<color rgba="0.117 0.117 0.117 1"/>
+		</material>
+	</visual>
+	<collision>
+		<origin xyz="0 0 0" rpy="${-3.1415927/2} 0 0"/>
+		<geometry>
+	    <!--mesh filename="package://amr_robots_description/meshes/p3at_meshes/wheel.stl"/-->
+	    <cylinder radius="0.111" length="0.075"/>
+		</geometry>
+	</collision>
+	</link>
+	<gazebo reference="p3at_front_${side}_wheel">
+		<material>Gazebo/Black</material>
+	</gazebo>
+	<joint name="p3at_front_${side}_wheel_joint" type="continuous">
+  	<axis xyz="0 1 0"/>
+    <anchor xyz="0 0 0"/>
+    <limit effort="100" velocity="100" />
+    <joint_properties damping="0.7"/>
+		<origin xyz="0 0 0" rpy="0 0 0"/>
+		<parent link="p3at_front_${side}_hub"/>
+		<child link="p3at_front_${side}_wheel"/>
+	</joint>
+<!-- Back Axles + Wheels + Hubcaps -->
+	<link name="p3at_back_${side}_axle">
+		<inertial>
+			<mass value="0.1"/>
+			<origin xyz="0 0 0"/>
+			<inertia ixx="1.0" ixy="0.0" ixz="0.0"
+				 iyy="1.0" iyz="0.0" izz="1.0"/>
+  	 	</inertial>
+	<visual>
+		<origin xyz="0 0 0" rpy="0 0 0"/>
+		<geometry>
+			<mesh filename="package://amr_robots_description/meshes/p3at_meshes/axle.stl"/>
+		</geometry>
+		<material name="AxleGrey">
+			<color rgba="0.5 0.5 0.5 1"/>
+		</material>
+	</visual>
+	<collision>
+		<origin xyz="0 0 0" rpy="0 0 0"/>
+		<geometry>
+			<mesh filename="package://amr_robots_description/meshes/p3at_meshes/axle.stl"/>
+		</geometry>
+	</collision>
+	</link>
+	<gazebo reference="p3at_back_${side}_axle">
+		<material value="Gazebo/Green"/>
+	</gazebo>
+	<joint name="p3at_back_${side}_axle_joint" type="fixed">
+		<origin xyz="-0.134 ${reflect*0.156} 0.111" rpy="0 0 0"/>
+		<parent link="base_link"/>
+		<child link="p3at_back_${side}_axle"/>
+	</joint>
+	<link name="p3at_back_${side}_hub">
+		<inertial>
+			<mass value="0.1"/>
+			<origin xyz="0 0 0"/>
+			<inertia ixx="1.0" ixy="0.0" ixz="0.0"
+				 iyy="1.0" iyz="0.0" izz="1.0"/>
+  	 	</inertial>
+	<visual name="base_visual">
+		<origin xyz="0 0 0" rpy="0 0 0"/>
+		<geometry name="pioneer_geom">
+			<mesh filename="package://amr_robots_description/meshes/p3at_meshes/${side}_hubcap.stl"/>
+		</geometry>
+		<material name="HubcapYellow"/>
+	</visual>
+	<collision>
+		<origin xyz="0 0 0" rpy="0 0 0"/>
+		<geometry>
+			<mesh filename="package://amr_robots_description/meshes/p3at_meshes/${side}_hubcap.stl"/>
+		</geometry>
+	</collision>
+	</link>
+	<gazebo reference="p3at_back_${side}_hub">
+		<material value="Gazebo/Yellow"/>
+	</gazebo>
+	<joint name="p3at_back_${side}_hub_joint" type="fixed">
+		<origin xyz="-0 ${reflect*0.041} 0" rpy="0 0 0"/>
+		<parent link="p3at_back_${side}_axle"/>
+		<child link="p3at_back_${side}_hub"/>
+	</joint>
+	<link name="p3at_back_${side}_wheel">
+		<inertial>
+			<mass value="1.2"/>
+			<origin xyz="0 0 0"/>
+			<inertia ixx="0.012411765597" ixy="0" ixz="0"
+                                                      iyy="0.015218160428" iyz="0"
+                                                                           izz="0.011763977943"/>
+      </inertial>
+	<visual>
+		<origin xyz="0 0 0" rpy="0 0 0"/>
+		<geometry>
+			<mesh filename="package://amr_robots_description/meshes/p3at_meshes/wheel.stl"/>
+		</geometry>
+	</visual>
+	<collision>
+		<origin xyz="0 0 0" rpy="${-3.1415927/2} 0 0"/>
+		<geometry>
+	    <!--mesh filename="package://amr_robots_description/meshes/p3at_meshes/wheel.stl"/-->
+	    <cylinder radius="0.111" length="0.075"/>
+		</geometry>
+	</collision>
+	</link>
+	<gazebo reference="p3at_back_${side}_wheel">
+		<material>Gazebo/Black</material>
+	</gazebo>
+	<joint name="p3at_back_${side}_wheel_joint" type="continuous">
+	  <axis xyz="0 1 0"/>
+    <anchor xyz="0 0 0"/>
+    <limit effort="100" velocity="100" />
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